Commit message: increase arm joint limits a bit for moveit

File: urdf/youbot_arm/arm.urdf.xacro (robot description, xacro)
@@ -47,5 +47,5 @@
 			<!-- damping - N*s/m, N*s*m/rad -->
 			<!-- friction - N, N*m -->
-			<limit effort="${9.5}" velocity="${M_PI / 2.0}" lower="0" upper="${joint_1_limit}"/>
+			<limit effort="${9.5}" velocity="${M_PI / 2.0}" lower="-0.01" upper="${joint_1_limit+0.01}"/>
 			<!--effort - N, N*m-->
 			<!--velocity - m/s, rad/s-->
@@ -84,5 +84,5 @@
 			<!--<calibration rising="${arm_2_ref}" falling="${arm_2_ref}"/>-->
 			<dynamics damping="1" friction="0.5" />
-			<limit effort="${9.5}" velocity="${M_PI / 2.0}" lower="0" upper="${joint_2_limit}"/>
+			<limit effort="${9.5}" velocity="${M_PI / 2.0}" lower="-0.01" upper="${joint_2_limit+0.01}"/>
       <!--safety_controller k_position="20" k_velocity="${2*9.5/M_PI}" soft_lower_limit="${threshold}" soft_upper_limit="${joint_2_limit_soft}" /-->
 		</joint>
@@ -123,5 +123,5 @@
 			<axis xyz="0 1 0"/>
 			<dynamics damping="1" friction="0.5" />
-			<limit effort="${6.0}" velocity="${M_PI / 2.0}" lower="-${joint_3_limit}" upper="0"/>
+			<limit effort="${6.0}" velocity="${M_PI / 2.0}" lower="-${joint_3_limit-0.01}" upper="0.01"/>
       <!--safety_controller k_position="20" k_velocity="50" soft_lower_limit="-${joint_3_limit_soft}" soft_upper_limit="-${threshold}" /-->
 		</joint>
@@ -155,5 +155,5 @@
 			<!--<calibration rising="${arm_4_ref}" falling="${arm_4_ref}"/>-->
 			<dynamics damping="1" friction="0.5" />
-			<limit effort="${2.0}" velocity="${M_PI / 2.0}" lower="0" upper="${joint_4_limit}"/>
+			<limit effort="${2.0}" velocity="${M_PI / 2.0}" lower="-0.01" upper="${joint_4_limit+0.01}"/>
 			<!--safety_controller k_position="20" k_velocity="100" soft_lower_limit="0" soft_upper_limit="${joint_4_limit_soft}" /-->
 		</joint>
@@ -187,5 +187,5 @@
 			<!--<calibration rising="${arm_5_ref}" falling="${arm_5_ref}"/>-->
 			<dynamics damping="0.5" friction="0.5" />
-			<limit effort="${1.0}" velocity="${M_PI / 2.0}" lower="0" upper="${joint_5_limit}" />
+			<limit effort="${1.0}" velocity="${M_PI / 2.0}" lower="-0.01" upper="${joint_5_limit+0.01}" />
       <!--safety_controller k_position="20" k_velocity="100" soft_lower_limit="0" soft_upper_limit="${joint_5_limit_soft}" /-->
 		</joint>
