Commit message: add basic moveit2+gazebo support

File: controller/ros_controller.urdf.xacro (robot description, xacro)
@@ -1,11 +1,54 @@
 <?xml version="1.0"?>
 <robot xmlns:sensor="http://playerstage.sourceforge.net/gazebo/xmlschema/#sensor"
-       xmlns:controller="http://playerstage.sourceforge.net/gazebo/xmlschema/#controller"
-       xmlns:interface="http://playerstage.sourceforge.net/gazebo/xmlschema/#interface">
+  xmlns:controller="http://playerstage.sourceforge.net/gazebo/xmlschema/#controller"
+  xmlns:interface="http://playerstage.sourceforge.net/gazebo/xmlschema/#interface">
   <gazebo>
-    <plugin name="gazebo_ros_controller" filename="libgazebo_ros_control.so">
-        <robotSimType>gazebo_ros_control/DefaultRobotHWSim</robotSimType>
-        <legacyModeNS>true</legacyModeNS>
+    <plugin filename="libgz_ros2_control-system.so"
+      name="gz_ros2_control::GazeboSimROS2ControlPlugin">
+      <parameters>$(find youbot_description)/controller/ros2_controllers.yaml</parameters>
     </plugin>
   </gazebo>
+  <plugin filename="libgz_ros2_control-system.so" name="gz_ros2_control::GazeboSimROS2ControlPlugin">
+    <parameters>$(find youbot_description)/controller/ros2_controllers.yaml</parameters>
+  </plugin>
+  <ros2_control name="gazebo_ros_controller" type="system">
+    <hardware>
+      <plugin>gz_ros2_control/GazeboSimSystem</plugin>
+    </hardware>
+    <joint name="arm_joint_1">
+      <command_interface name="position" />
+      <state_interface name="position">
+        <param name="initial_value">0</param>
+      </state_interface>
+      <state_interface name="velocity" />
+    </joint>
+    <joint name="arm_joint_2">
+      <command_interface name="position" />
+      <state_interface name="position">
+        <param name="initial_value">0</param>
+      </state_interface>
+      <state_interface name="velocity" />
+    </joint>
+    <joint name="arm_joint_3">
+      <command_interface name="position" />
+      <state_interface name="position">
+        <param name="initial_value">0</param>
+      </state_interface>
+      <state_interface name="velocity" />
+    </joint>
+    <joint name="arm_joint_4">
+      <command_interface name="position" />
+      <state_interface name="position">
+        <param name="initial_value">0</param>
+      </state_interface>
+      <state_interface name="velocity" />
+    </joint>
+    <joint name="arm_joint_5">
+      <command_interface name="position" />
+      <state_interface name="position">
+        <param name="initial_value">0</param>
+      </state_interface>
+      <state_interface name="velocity" />
+    </joint>
+  </ros2_control>
 </robot>

File: urdf/youbot_base/base.gazebo.xacro (robot description, xacro)
@@ -1,7 +1,8 @@
 <?xml version="1.0"?>
 <robot xmlns:sensor="http://playerstage.sourceforge.net/gazebo/xmlschema/#sensor"
-       xmlns:controller="http://playerstage.sourceforge.net/gazebo/xmlschema/#controller"
-       xmlns:interface="http://playerstage.sourceforge.net/gazebo/xmlschema/#interface"
-       xmlns:xacro="http://www.ros.org/wiki/xacro/#interface">
+  xmlns:controller="http://playerstage.sourceforge.net/gazebo/xmlschema/#controller"
+  xmlns:interface="http://playerstage.sourceforge.net/gazebo/xmlschema/#interface"
+  xmlns:gz="http://playerstage.sourceforge.net/gazebo/xmlschema"
+  xmlns:xacro="http://www.ros.org/wiki/xacro/#interface">
   <xacro:macro name="youbot_base_gazebo">
     <gazebo reference="youbot_base">
@@ -9,29 +10,76 @@
     <!-- front left wheel -->
     <gazebo reference="wheel_link_fl">
-      <kp>1000000</kp>
-      <kd>100</kd>
-    </gazebo>
-    <gazebo reference="caster_link_fl">
+      <collision>
+        <surface>
+          <friction>
+            <ode>
+              <mu>1.0</mu>
+              <mu2>0.0</mu2>
+              <fdir1 gz:expressed_in="base_footprint">1 -1 0</fdir1>
+            </ode>
+          </friction>
+        </surface>
+      </collision>
     </gazebo>
     <!-- front right wheel -->
     <gazebo reference="wheel_link_fr">
-      <kp>1000000</kp>
-      <kd>100</kd>
-    </gazebo>
-    <gazebo reference="caster_link_fr">
+      <collision>
+        <surface>
+          <friction>
+            <ode>
+              <mu>1.0</mu>
+              <mu2>0.0</mu2>
+              <fdir1 gz:expressed_in="base_footprint">1 1 0</fdir1>
+            </ode>
+          </friction>
+        </surface>
+      </collision>
     </gazebo>
     <!-- back left wheel -->
     <gazebo reference="wheel_link_bl">
-      <kp>1000000</kp>
-      <kd>100</kd>
-    </gazebo>
-    <gazebo reference="caster_link_bl">
+      <collision>
+        <surface>
+          <friction>
+            <ode>
+              <mu>1.0</mu>
+              <mu2>0.0</mu2>
+              <fdir1 gz:expressed_in="base_footprint">1 1 0</fdir1>
+            </ode>
+          </friction>
+        </surface>
+      </collision>
     </gazebo>
     <!-- back right wheel -->
     <gazebo reference="wheel_link_br">
-      <kp>1000000</kp>
-      <kd>100</kd>
+      <collision>
+        <surface>
+          <friction>
+            <ode>
+              <mu>1.0</mu>
+              <mu2>0.0</mu2>
+              <fdir1 gz:expressed_in="base_footprint">1 -1 0</fdir1>
+            </ode>
+          </friction>
+        </surface>
+      </collision>
     </gazebo>
-    <gazebo reference="caster_link_br">
+    <gazebo>
+      <plugin
+        filename="gz-sim-joint-state-publisher-system"
+        name="gz::sim::systems::JointStatePublisher">
+      </plugin>
+      <plugin filename="gz-sim-mecanum-drive-system" name="gz::sim::systems::MecanumDrive">
+        <front_left_joint>wheel_joint_fl</front_left_joint>
+        <front_right_joint>wheel_joint_fr</front_right_joint>
+        <back_left_joint>wheel_joint_bl</back_left_joint>
+        <back_right_joint>wheel_joint_br</back_right_joint>
+        <wheelbase>0.45</wheelbase>
+        <wheel_separation>0.3</wheel_separation>
+        <wheel_radius>0.0475</wheel_radius>
+        <min_acceleration>-5</min_acceleration>
+        <max_acceleration>5</max_acceleration>
+        <frame_id>odom</frame_id>
+        <child_frame_id>base_footprint</child_frame_id>
+      </plugin>
     </gazebo>
   </xacro:macro>

File: urdf/youbot_plate/plate.urdf.xacro (robot description, xacro)
@@ -22,5 +22,5 @@
 					<mesh filename="package://youbot_description/meshes/youbot_plate/plate.dae" />
 				</geometry>
-				<material name="DarkGrey"/>
+				<material name="youbot/DarkGrey"/>
 			</visual>
 			<collision>
